File: PCB/Simple_Sprouts_PCB/Simple_Sprouts_PCB.kicad_sch (KiCad schematic)
At the start: 38 parts, among them J1 Raspberry_Pi_5, J3 Soil Sensor, J4 Soil Sensor, J5 Water Level Sensor, J6 Temperature Sensor, J7 Air Quality Sensor, J8 Humidity Sensor, J9 Fan, Q1 NMOS, Q2 NMOS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

Commit message: Add files via upload
Parts:
- Q1, Q2, Q3, Q4, Q5, Q6: value NMOS -> IRLB8721PbF
- R10, R11, R12, R13: value 600Ω -> 5kΩ
- R2, R3: value 10kΩ -> 4.7kΩ
Connections:
- net +12V: now also D1.2 (A), D2.2 (A), D3.2 (A), D4.2 (A); no longer D1.1 (K), D2.1 (K), D3.1 (K), D4.1 (K)
- net +5V: now also LEDStrip1.-, LEDStrip2.-; no longer LEDStrip1.+, LEDStrip2.+, R2.2, R3.2
- net at Q2.2 (D): now also LEDStrip2.+; no longer LEDStrip2.-
- net at J1.3 (SDA_I2C1/GPIO02), J3.3 (Pin_3), J4.3 (Pin_3)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: now also J1.5 (SCL_I2C1/GPIO03), J3.4 (Pin_4), J4.4 (Pin_4), J6.4 (Pin_4), J7.4 (Pin_4), J8.4 (Pin_4), R3.1, U4.5 (SCL)
- net at R11.1: now also D2.1 (K); no longer D2.2 (A)
- net at R13.1: now also D4.1 (K); no longer D4.2 (A)
- net at Q3.2 (D): now also LEDStrip1.+; no longer LEDStrip1.-
- net at R10.1: now also D1.1 (K); no longer D1.2 (A)
- net at R12.1: now also D3.1 (K); no longer D3.2 (A)
- new net +3.3V: R2.2, R3.2
Other:
- moved on the sheet: Adafruit_Solenoid_Valve1, D1, D2, D3, D4, J3, J4, J6, J7, J8, LEDStrip1A, LEDStrip2A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

Commit message: Add files via upload
Parts:
- added J10: NoIR Camera Module, symbol Connector_Generic:Conn_01x01
Connections:
- net at J1.3 (SDA_I2C1/GPIO02), J3.3 (Pin_3), J4.3 (Pin_3)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: no longer J1.5 (SCL_I2C1/GPIO03), J3.4 (Pin_4), J4.4 (Pin_4), J6.4 (Pin_4), J7.4 (Pin_4), J8.4 (Pin_4), R3.1, U4.5 (SCL)
- new net: J1.5 (SCL_I2C1/GPIO03), J3.4 (Pin_4), J4.4 (Pin_4), J6.4 (Pin_4), J7.4 (Pin_4), J8.4 (Pin_4), R3.1, U4.5 (SCL)
- new net: J1.y (Camera), J10.1 (Pin_1)

Commit message: Add files via upload
Parts:
- removed J5: Water Level Sensor, symbol Connector_Generic:Conn_01x03
- removed U1: CRE1S0505DC, Converter_DCDC:Converter_DCDC_Murata_CRE1xxxxxxDC_THT, symbol Regulator_Switching:CRE1S0505DC
- removed U4: ADC101C021CIMK, Package_TO_SOT_SMD:SOT-23-6, symbol Analog_ADC:ADC101C021CIMK
- added D5, D6, D7, D8: SR5100, symbol Device:D_Schottky
- added J9: HC-SR04, symbol Connector_Generic:Conn_01x04
- added R14: 1kΩ, symbol Device:R
- added R15: 2kΩ, symbol Device:R
- added U1, U2: DC-DC Converter, symbol Converter_DCDC:TME-0305S
- R4, R5, R6, R7, R8, R9: value 10kΩ -> 220Ω
- renumbered Adafruit_Solenoid_Valve to Solenoid_Valve, Adafruit_Solenoid_Valve1 to Solenoid_Valve
Connections:
- net +12V: now also D5.2 (A), D6.2 (A), D7.2 (A), D8.2 (A), U1.4 (+Vout)
- net +3.3V: now also J1.1 (3V3), J1.17 (3V3)
- net +5V: now also J9.1 (Pin_1), U2.4 (+Vout)
- net GND: now also J9.4 (Pin_4), R15.2, U1.1 (-Vin), U1.3 (-Vout), U2.1 (-Vin), U2.3 (-Vout)
- net at Q6.2 (D), R13.2, WaterPump1.2 (-): now also D7.1 (K)
- net at Q5.2 (D), Solenoid_Valve.2: now also R11.2, D6.1 (K)
- net at Q1.2 (D), R1.2, R12.2: now also D8.1 (K)
- net at Q4.2 (D), Solenoid_Valve.2: now also R10.2, D5.1 (K)
- net at J1.29 (GPCLK1/GPIO05): now also R14.1, R15.1
- net at J1.7 (GPCLK0/GPIO04): now also J9.2 (Pin_2)
- new net: J9.3 (Pin_3), R14.2
- new net +24V: U1.2 (+Vin), U2.2 (+Vin)
Other:
- moved on the sheet: R8

Commit message: Add files via upload
Parts:
- renumbered J9 to J11, Solenoid_Valve to Solenoid_Valve1, Solenoid_Valve to Solenoid_Valve2
Changed lines of the file:
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@@
 		(on_board yes)
 		(dnp no)
-		(property "Reference" "Solenoid_Valve"
+		(property "Reference" "Solenoid_Valve2"
 			(at 88.9 94.742 90)
 			(effects
@@
 			(project ""
 				(path "/a5df5b5c-9e14-4fe1-8dcb-bdc183e40462"
-					(reference "Solenoid_Valve")
+					(reference "Solenoid_Valve2")
 					(unit 1)
 				)
@@
 		(on_board yes)
 		(dnp no)
-		(property "Reference" "J9"
+		(property "Reference" "J11"
 			(at 169.926 61.468 90)
 			(effects
@@
 			(project ""
 				(path "/a5df5b5c-9e14-4fe1-8dcb-bdc183e40462"
-					(reference "J9")
+					(reference "J11")
 					(unit 1)
 				)
@@
 		(on_board yes)
 		(dnp no)
-		(property "Reference" "Solenoid_Valve"
+		(property "Reference" "Solenoid_Valve1"
 			(at 46.228 94.996 90)
 			(effects
@@
 			(project "Simple_Sprouts_PCB"
 				(path "/a5df5b5c-9e14-4fe1-8dcb-bdc183e40462"
-					(reference "Solenoid_Valve")
+					(reference "Solenoid_Valve1")
 					(unit 1)
 				)

Commit message: Add files via upload
Parts:
- D5, D6, D7, D8: value SR5100 -> SS510
Connections:
- net at Q6.2 (D), R13.2, WaterPump1.2 (-): now also D8.1 (K); no longer D7.1 (K)
- net at Q1.2 (D), R1.2, R12.2: now also D7.1 (K); no longer D8.1 (K)

Commit message: Add files via upload
Parts:
- D1, D2, D3, D4: footprint (none) -> my-LED-4mm-3mm:LED_D4.0mm_P3.0mm
- D5, D6, D7, D8: footprint (none) -> Diode_SMD:D_SMB
- J1: footprint (none) -> RASPBERRY_PI_4B_4GB:MODULE_RASPBERRY_PI_4B_4GB
- J3, J4: footprint (none) -> No_Footprint:No_Footprint
- R10, R11, R12, R13, R2, R3: footprint (none) -> Resistor_SMD:R_0805_2012Metric
- R14: footprint (none) -> Resistor_SMD:R_1210_3225Metric
- R15: footprint (none) -> Resistor_SMD:R_2512_6332Metric
- R4, R5, R6, R7, R8, R9: footprint (none) -> Resistor_SMD:R_1206_3216Metric
Connections:
- net +3.3V: now also R2.1; no longer R2.2
- net at J1.3 (SDA_I2C1/GPIO02), J3.3 (Pin_3), J4.3 (Pin_3)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: now also R2.2; no longer R2.1
- net at J1.13 (GPIO27/SDIO_DAT3), Q1.1 (G): now also R7.1; no longer R4.1
- net at J1.37 (GPIO26/SDIO_DAT2), Q2.1 (G): now also R6.1; no longer R5.1
- net at J1.22 (GPIO25/SDIO_DAT1), Q3.1 (G): now also R5.1; no longer R6.1
- net at J1.33 (GPIO13/PWM1), Q5.1 (G): now also R4.1; no longer R7.1

Commit message: Add files via upload
Parts:
- J1: footprint RASPBERRY_PI_4B_4GB:MODULE_RASPBERRY_PI_4B_4GB -> RASPBERRY_PI_4B_4GB:Pin_Replacement
Connections:
- net at Q1.1 (G), R7.1: now also J1.19 (MOSI_SPI0/GPIO10); no longer J1.13 (GPIO27/SDIO_DAT3)
- net at Q6.1 (G), R9.1: now also J1.27 (ID_SD_I2C0/GPIO00); no longer J1.23 (SCLK_SPI0/GPIO11)
- net at Q4.1 (G), R8.1: now also J1.33 (GPIO13/PWM1); no longer J1.32 (GPIO12/PWM0)
- net at R14.1, R15.1: now also J1.13 (GPIO27/SDIO_DAT3); no longer J1.29 (GPCLK1/GPIO05)
- net at Q2.1 (G), R6.1: now also J1.11 (GPIO17/SPI1_~{CE1}); no longer J1.37 (GPIO26/SDIO_DAT2)
- net at Q5.1 (G), R4.1: now also J1.35 (GPIO19/SPI1_MISO/PCM_FS); no longer J1.33 (GPIO13/PWM1)
- net at J1.15 (GPIO22/SDIO_CLK): now also Q3.1 (G), R5.1
- net at J1.16 (GPIO23/SDIO_CMD): now also J9.2 (Pin_2)
- net at J1.7 (GPCLK0/GPIO04): no longer J9.2 (Pin_2)
- now unconnected: J1.22 (GPIO25/SDIO_DAT1)
Other:
- moved on the sheet: D3, D4, D7, D8, J9, LEDStrip1A, LEDStrip2A, Q1, Q2, Q3, Q6, R12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

Commit message: Add files via upload
Parts:
- added J2: Screw_Terminal, FootprintsLibrary:MyTerminalBlock_MaiXu_MX126-5.0-04P_1x04_P5.00mm, symbol Connector:Screw_Terminal_01x04
Other:
- moved on the sheet: U2
Changed lines of the file:
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@@
 	(wire
 		(pts
-			(xy 124.46 53.34) (xy 125.73 53.34)
+			(xy 160.02 39.37) (xy 161.29 39.37)
 		)
 		(stroke
@@
 	(wire
 		(pts
+			(xy 120.65 53.34) (xy 113.03 53.34)
+		)
+		(stroke
+			(width 0)
+			(type default)
+		)
+	)
+	(wire
+		(pts
 			(xy 271.78 88.9) (xy 274.32 88.9)
 		)
@@
 	(wire
 		(pts
-			(xy 147.32 53.34) (xy 146.05 53.34)
+			(xy 182.88 39.37) (xy 181.61 39.37)
 		)
 		(stroke
@@
 	(wire
 		(pts
+			(xy 119.38 54.61) (xy 119.38 58.42)
+		)
+		(stroke
+			(width 0)
+			(type default)
+		)
+	)
+	(wire
+		(pts
 			(xy 260.35 60.96) (xy 260.35 88.9)
 		)
@@
 	(wire
 		(pts
+			(xy 119.38 58.42) (xy 113.03 58.42)
+		)
+		(stroke
+			(width 0)
+			(type default)
+		)
+	)
+	(wire
+		(pts
 			(xy 49.53 86.36) (xy 55.88 86.36)
 		)
@@
 	(wire
 		(pts
+			(xy 125.73 54.61) (xy 119.38 54.61)
+		)
+		(stroke
+			(width 0)
+			(type default)
+		)
+	)
+	(wire
+		(pts
 			(xy 158.75 125.73) (xy 158.75 148.59)
 		)
@@
 	(wire
 		(pts
+			(xy 120.65 52.07) (xy 120.65 53.34)
+		)
+		(stroke
+			(width 0)
+			(type default)
+		)
+	)
+	(wire
+		(pts
 			(xy 260.35 88.9) (xy 264.16 88.9)
 		)
@@
 	(wire
 		(pts
-			(xy 114.3 53.34) (xy 113.03 53.34)
+			(xy 125.73 52.07) (xy 120.65 52.07)
 		)
 		(stroke
@@
 	(symbol
 		(lib_id "power:GND")
-		(at 113.03 58.42 0)
+		(at 125.73 54.61 90)
 		(unit 1)
 		(exclude_from_sim no)
@@
 		(on_board yes)
 		(dnp no)
-		(fields_autoplaced yes)
 		(property "Reference" "#PWR041"
-			(at 113.03 64.77 0)
+			(at 132.08 54.61 0)
 			(effects
 				(font
@@
 		)
 		(property "Value" "GND"
-			(at 113.03 63.5 0)
+			(at 122.936 56.388 90)
 			(effects
 				(font
 					(size 1.27 1.27)
 				)
+				(justify right)
 			)
 		)
 		(property "Footprint" ""
-			(at 113.03 58.42 0)
+			(at 125.73 54.61 0)
 			(effects
 				(font
@@
 		)
 		(property "Datasheet" ""
-			(at 113.03 58.42 0)
+			(at 125.73 54.61 0)
 			(effects
 				(font
@@
 		)
 		(property "Description" "Power symbol creates a global label with name \"GND\" , ground"
-			(at 113.03 58.42 0)
+			(at 125.73 54.61 0)
 			(effects
 				(font
@@
 	)
 	(symbol
+		(lib_id "Connector:Screw_Terminal_01x04")
+		(at 133.35 54.61 0)
+		(unit 1)
+		(exclude_from_sim no)
+		(in_bom yes)
+		(on_board yes)
+		(dnp no)
+		(fields_autoplaced yes)
+		(property "Reference" "J2"
+			(at 135.89 54.6099 0)
+			(effects
+				(font
+					(size 1.27 1.27)
+				)
+				(justify left)
+			)
+		)
+		(property "Value" "Screw_Terminal"
+			(at 135.89 57.1499 0)
+			(effects
+				(font
+					(size 1.27 1.27)
+				)
+				(justify left)
+			)
+		)
+		(property "Footprint" "FootprintsLibrary:MyTerminalBlock_MaiXu_MX126-5.0-04P_1x04_P5.00mm"
+			(at 133.35 54.61 0)
+			(effects
+				(font
+					(size 1.27 1.27)
+				)
+				(hide yes)
+			)
+		)
+		(property "Datasheet" "~https://www.lcsc.com/datasheet/lcsc_datasheet_2109030930_HIWA-PA001-4P_C173286.pdf"
+			(at 133.35 54.61 0)
+			(effects
+				(font
+					(size 1.27 1.27)
+				)
+				(hide yes)
+			)
+		)
+		(property "Description" "Generic screw terminal, single row, 01x04, script generated (kicad-library-utils/schlib/autogen/connector/)"
+			(at 133.35 54.61 0)
+			(effects
+				(font
+					(size 1.27 1.27)
+				)
+				(hide yes)
+			)
+		)
+		(pin "1"
+		)
+		(pin "2"
+		)
+		(pin "4"
+		)
+		(pin "3"
+		)
+		(instances
+			(project ""
+				(path "/a5df5b5c-9e14-4fe1-8dcb-bdc183e40462"
+					(reference "J2")
+					(unit 1)
+				)
+			)
+		)
+	)
+	(symbol
 		(lib_id "power:GND")
 		(at 217.17 124.46 0)
@@
 	(symbol
 		(lib_id "Converter_DCDC:TME-0305S")
-		(at 135.89 55.88 0)
+		(at 171.45 41.91 0)
 		(unit 1)
 		(exclude_from_sim no)
@@
 		(fields_autoplaced yes)
 		(property "Reference" "U2"
-			(at 135.89 45.72 0)
+			(at 171.45 31.75 0)
 			(effects
 				(font
@@
 		)
 		(property "Value" "DC-DC Converter"
-			(at 135.89 48.26 0)
+			(at 171.45 34.29 0)
 			(effects
 				(font
@@
 		)
 		(property "Footprint" ""
-			(at 135.89 64.77 0)
+			(at 171.45 50.8 0)
 			(effects
 				(font
@@
 		)
 		(property "Datasheet" "https://www.amazon.com/gp/product/B0CRVW7N2J/ref=ox_sc_act_image_1?smid=A1QRG6NHEUKUZO&th=1"
-			(at 135.89 62.23 0)
+			(at 171.45 48.26 0)
 			(effects
 				(font
@@
 		)
 		(property "Description" "DC 12V/24V to 5V USB C Step Down Converter Type-C Interface 5A 25W Waterproof Buck Module Power Adapter"
-			(at 135.89 55.88 0)
+			(at 171.45 41.91 0)
 			(effects
 				(font
@@
 	(symbol
 		(lib_id "power:+12V")
-		(at 114.3 53.34 0)
+		(at 125.73 52.07 270)
 		(unit 1)
 		(exclude_from_sim no)
@@
 		(on_board yes)
 		(dnp no)
-		(fields_autoplaced yes)
 		(property "Reference" "#PWR040"
-			(at 114.3 57.15 0)
+			(at 121.92 52.07 0)
 			(effects
 				(font
@@
 		)
 		(property "Value" "+12V"
-			(at 114.3 48.26 0)
+			(at 121.412 50.038 90)
 			(effects
 				(font
 					(size 1.27 1.27)
 				)
+				(justify left)
 			)
 		)
 		(property "Footprint" ""
-			(at 114.3 53.34 0)
+			(at 125.73 52.07 0)
 			(effects
 				(font
@@
 		)
 		(property "Datasheet" ""
-			(at 114.3 53.34 0)
+			(at 125.73 52.07 0)
 			(effects
 				(font
@@
 		)
 		(property "Description" "Power symbol creates a global label with name \"+12V\""
-			(at 114.3 53.34 0)
+			(at 125.73 52.07 0)
 			(effects
 				(font
@@
 	(symbol
 		(lib_id "power:GND")
-		(at 146.05 58.42 0)
+		(at 181.61 44.45 0)
 		(unit 1)
 		(exclude_from_sim no)
@@
 		(fields_autoplaced yes)
 		(property "Reference" "#PWR045"
-			(at 146.05 64.77 0)
+			(at 181.61 50.8 0)
 			(effects
 				(font
@@
 		)
 		(property "Value" "GND"
-			(at 146.05 63.5 0)
+			(at 181.61 49.53 0)
 			(effects
 				(font
@@
 		)
 		(property "Footprint" ""
-			(at 146.05 58.42 0)
+			(at 181.61 44.45 0)
 			(effects
 				(font
@@
 		)
 		(property "Datasheet" ""
-			(at 146.05 58.42 0)
+			(at 181.61 44.45 0)
 			(effects
 				(font
@@
 		)
 		(property "Description" "Power symbol creates a global label with name \"GND\" , ground"
-			(at 146.05 58.42 0)
+			(at 181.61 44.45 0)
 			(effects
 				(font
@@
 	(symbol
 		(lib_id "power:GND")
-		(at 125.73 58.42 0)
+		(at 161.29 44.45 0)
 		(unit 1)
 		(exclude_from_sim no)
@@
 		(fields_autoplaced yes)
 		(property "Reference" "#PWR044"
-			(at 125.73 64.77 0)
+			(at 161.29 50.8 0)
 			(effects
 				(font
@@
 		)
 		(property "Value" "GND"
-			(at 125.73 63.5 0)
+			(at 161.29 49.53 0)
 			(effects
 				(font
@@
 		)
 		(property "Footprint" ""
-			(at 125.73 58.42 0)
+			(at 161.29 44.45 0)
 			(effects
 				(font
@@
 		)
 		(property "Datasheet" ""
-			(at 125.73 58.42 0)
+			(at 161.29 44.45 0)
 			(effects
 				(font
@@
 		)
 		(property "Description" "Power symbol creates a global label with name \"GND\" , ground"
-			(at 125.73 58.42 0)
+			(at 161.29 44.45 0)
 			(effects
 				(font
@@
 	(symbol
 		(lib_id "power:+24V")
-		(at 124.46 53.34 0)
+		(at 160.02 39.37 0)
 		(unit 1)
 		(exclude_from_sim no)
@@
 		(fields_autoplaced yes)
 		(property "Reference" "#PWR043"
-			(at 124.46 57.15 0)
+			(at 160.02 43.18 0)
 			(effects
 				(font
@@
 		)
 		(property "Value" "+24V"
-			(at 124.46 48.26 0)
+			(at 160.02 34.29 0)
 			(effects
 				(font
@@
 		)
 		(property "Footprint" ""
-			(at 124.46 53.34 0)
+			(at 160.02 39.37 0)
 			(effects
 				(font
@@
 		)
 		(property "Datasheet" ""
-			(at 124.46 53.34 0)
+			(at 160.02 39.37 0)
 			(effects
 				(font
@@
 		)
 		(property "Description" "Power symbol creates a global label with name \"+24V\""
-			(at 124.46 53.34 0)
+			(at 160.02 39.37 0)
 			(effects
 				(font
@@
 	(symbol
 		(lib_id "power:+12V")
-		(at 147.32 53.34 0)
+		(at 182.88 39.37 0)
 		(unit 1)
 		(exclude_from_sim no)
@@
 		(fields_autoplaced yes)
 		(property "Reference" "#PWR047"
-			(at 147.32 57.15 0)
+			(at 182.88 43.18 0)
 			(effects
 				(font
@@
 		)
 		(property "Value" "+5V"
-			(at 147.32 48.26 0)
+			(at 182.88 34.29 0)
 			(effects
 				(font
@@
 		)
 		(property "Footprint" ""
-			(at 147.32 53.34 0)
+			(at 182.88 39.37 0)
 			(effects
 				(font
@@
 		)
 		(property "Datasheet" ""
-			(at 147.32 53.34 0)
+			(at 182.88 39.37 0)
 			(effects
 				(font
@@
 		)
 		(property "Description" "Power symbol creates a global label with name \"+12V\""
-			(at 147.32 53.34 0)
+			(at 182.88 39.37 0)
 			(effects
 				(font
