File: PCB/Simple_Sprouts_PCB/Simple_Sprouts_PCB.kicad_sch (KiCad schematic)
At the start: 46 parts, among them J1 Raspberry_Pi_5, J10 NoIR Camera Module, J11 Fan, J2 Screw_Terminal, J3 Soil Sensor, J4 Soil Sensor, J6 Temperature Sensor, J7 Air Quality Sensor, J8 Humidity Sensor, J9 HC-SR04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

Commit message: Add files via upload
Parts:
- removed J2: Screw_Terminal, FootprintsLibrary:MyTerminalBlock_MaiXu_MX126-5.0-04P_1x04_P5.00mm, symbol Connector:Screw_Terminal_01x04
- R4, R5, R6, R7, R8, R9: value 220Ω -> 10kΩ
Connections:
- net +12V: now also D5.1 (K), D6.1 (K), D7.1 (K), D8.1 (K); no longer D5.2 (A), D6.2 (A), D7.2 (A), D8.2 (A)
- net at Q6.2 (D), R13.2, WaterPump1.2 (-): now also D8.2 (A); no longer D8.1 (K)
- net at Q5.2 (D), R11.2, Solenoid_Valve2.2: now also D6.2 (A); no longer D6.1 (K)
- net at Q1.2 (D), R1.2, R12.2: now also D7.2 (A); no longer D7.1 (K)
- net at Q4.2 (D), R10.2, Solenoid_Valve1.2: now also D5.2 (A); no longer D5.1 (K)
Other:
- moved on the sheet: D5, D6, D7, D8, U1, U2

Commit message: Add files via upload
Parts:
- J3, J4: footprint No_Footprint:No_Footprint -> Connector_PinHeader_2.54mm:PinHeader_1x04_P2.54mm_Vertical
- J6, J7, J8, J9: footprint (none) -> Connector_PinHeader_2.54mm:PinHeader_1x04_P2.54mm_Vertical
- LEDStrip1, LEDStrip2: footprint Display:HDSP-4840 -> TerminalBlock_Phoenix:TerminalBlock_Phoenix_MPT-0,5-2-2.54_1x02_P2.54mm_Horizontal
- R1, Solenoid_Valve1, Solenoid_Valve2, WaterPump1: footprint (none) -> TerminalBlock_Phoenix:TerminalBlock_Phoenix_MPT-0,5-2-2.54_1x02_P2.54mm_Horizontal
Changed lines of the file:
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@@
 		(exclude_from_sim no)
 		(in_bom yes)
-		(on_board no)
+		(on_board yes)
 		(dnp no)
 		(property "Reference" "LEDStrip2"
@@
 			)
 		)
-		(property "Footprint" "Display:HDSP-4840"
+		(property "Footprint" "TerminalBlock_Phoenix:TerminalBlock_Phoenix_MPT-0,5-2-2.54_1x02_P2.54mm_Horizontal"
 			(at 38.1 129.54 0)
 			(effects
@@
 		(exclude_from_sim no)
 		(in_bom yes)
-		(on_board no)
+		(on_board yes)
 		(dnp no)
 		(property "Reference" "J8"
@@
 			)
 		)
-		(property "Footprint" ""
+		(property "Footprint" "Connector_PinHeader_2.54mm:PinHeader_1x04_P2.54mm_Vertical"
 			(at 257.81 55.88 0)
 			(effects
@@
 		(exclude_from_sim no)
 		(in_bom yes)
-		(on_board no)
+		(on_board yes)
 		(dnp no)
 		(property "Reference" "J4"
@@
 			)
 		)
-		(property "Footprint" "No_Footprint:No_Footprint"
+		(property "Footprint" "Connector_PinHeader_2.54mm:PinHeader_1x04_P2.54mm_Vertical"
 			(at 219.71 55.88 0)
 			(effects
@@
 		(exclude_from_sim no)
 		(in_bom yes)
-		(on_board no)
+		(on_board yes)
 		(dnp no)
 		(property "Reference" "WaterPump1"
@@
 			)
 		)
-		(property "Footprint" ""
+		(property "Footprint" "TerminalBlock_Phoenix:TerminalBlock_Phoenix_MPT-0,5-2-2.54_1x02_P2.54mm_Horizontal"
 			(at 217.17 108.966 0)
 			(effects
@@
 		(exclude_from_sim no)
 		(in_bom yes)
-		(on_board no)
+		(on_board yes)
 		(dnp no)
 		(property "Reference" "Solenoid_Valve2"
@@
 			)
 		)
-		(property "Footprint" ""
+		(property "Footprint" "TerminalBlock_Phoenix:TerminalBlock_Phoenix_MPT-0,5-2-2.54_1x02_P2.54mm_Horizontal"
 			(at 91.44 90.17 0)
 			(effects
@@
 		(exclude_from_sim no)
 		(in_bom yes)
-		(on_board no)
+		(on_board yes)
 		(dnp no)
 		(property "Reference" "J3"
@@
 			)
 		)
-		(property "Footprint" "No_Footprint:No_Footprint"
+		(property "Footprint" "Connector_PinHeader_2.54mm:PinHeader_1x04_P2.54mm_Vertical"
 			(at 207.01 55.88 0)
 			(effects
@@
 		(exclude_from_sim no)
 		(in_bom yes)
-		(on_board no)
+		(on_board yes)
 		(dnp no)
 		(property "Reference" "LEDStrip1"
@@
 			)
 		)
-		(property "Footprint" "Display:HDSP-4840"
+		(property "Footprint" "TerminalBlock_Phoenix:TerminalBlock_Phoenix_MPT-0,5-2-2.54_1x02_P2.54mm_Horizontal"
 			(at 85.09 127 0)
 			(effects
@@
 		(on_board yes)
 		(dnp no)
-		(fields_autoplaced yes)
 		(property "Reference" "J1"
-			(at 154.94 66.04 0)
+			(at 146.558 69.342 0)
 			(effects
 				(font
 					(size 1.27 1.27)
 				)
+				(justify left)
 			)
 		)
 		(property "Value" "Raspberry_Pi_5"
-			(at 154.94 68.58 0)
+			(at 152.146 69.342 0)
 			(effects
 				(font
 					(size 1.27 1.27)
 				)
+				(justify left)
 			)
 		)
@@
 		(exclude_from_sim no)
 		(in_bom yes)
-		(on_board no)
+		(on_board yes)
 		(dnp no)
 		(property "Reference" "J7"
@@
 			)
 		)
-		(property "Footprint" ""
+		(property "Footprint" "Connector_PinHeader_2.54mm:PinHeader_1x04_P2.54mm_Vertical"
 			(at 245.11 55.88 0)
 			(effects
@@
 		(exclude_from_sim no)
 		(in_bom yes)
-		(on_board no)
+		(on_board yes)
 		(dnp no)
 		(property "Reference" "R1"
@@
 			)
 		)
-		(property "Footprint" ""
+		(property "Footprint" "TerminalBlock_Phoenix:TerminalBlock_Phoenix_MPT-0,5-2-2.54_1x02_P2.54mm_Horizontal"
 			(at 168.402 139.7 90)
 			(effects
@@
 		(exclude_from_sim no)
 		(in_bom yes)
-		(on_board no)
+		(on_board yes)
 		(dnp no)
 		(property "Reference" "Solenoid_Valve1"
@@
 			)
 		)
-		(property "Footprint" ""
+		(property "Footprint" "TerminalBlock_Phoenix:TerminalBlock_Phoenix_MPT-0,5-2-2.54_1x02_P2.54mm_Horizontal"
 			(at 49.53 90.17 0)
 			(effects
@@
 		(exclude_from_sim no)
 		(in_bom yes)
-		(on_board no)
+		(on_board yes)
 		(dnp no)
 		(property "Reference" "J6"
@@
 			)
 		)
-		(property "Footprint" ""
+		(property "Footprint" "Connector_PinHeader_2.54mm:PinHeader_1x04_P2.54mm_Vertical"
 			(at 232.41 55.88 0)
 			(effects
@@
 		(exclude_from_sim no)
 		(in_bom yes)
-		(on_board no)
+		(on_board yes)
 		(dnp no)
 		(fields_autoplaced yes)
@@
 			)
 		)
-		(property "Footprint" ""
+		(property "Footprint" "Connector_PinHeader_2.54mm:PinHeader_1x04_P2.54mm_Vertical"
 			(at 128.27 139.7 0)
 			(effects

Commit message: Add files via upload
Parts:
- added J2: 12V IN, Connector_PinHeader_2.00mm:PinHeader_1x01_P2.00mm_Vertical, symbol Connector_Generic:Conn_01x01
- added J5: 5V IN, Connector_PinHeader_2.00mm:PinHeader_1x01_P2.00mm_Vertical, symbol Connector_Generic:Conn_01x01
- J1: footprint RASPBERRY_PI_4B_4GB:Pin_Replacement -> RASPBERRY_PI_4B_4GB:RPI Pins
- R1: value Heater Module -> Heater
- renumbered LEDStrip1 to GROW1, LEDStrip2 to GROW2, Solenoid_Valve1 to Valve1, Solenoid_Valve2 to Valve2, WaterPump1 to Water_Pump1
Connections:
- net +12V: now also J2.1 (Pin_1)
- net +5V: now also J5.1 (Pin_1)
