File: PCB/Simple_Sprouts_PCB/Simple_Sprouts_PCB.kicad_sch (KiCad schematic)
At the start: 47 parts, among them J1 Raspberry_Pi_5, J10 NoIR Camera Module, J11 Fan, J12 12V, J2 12V IN, J3 Soil Sensor, J4 Soil Sensor, J5 5V IN, J6 Temperature Sensor, J7 Air Quality Sensor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

Commit message: Add files via upload
Connections:
- net +5V: now also GROW1.2, GROW2.2; no longer GROW1.-, GROW2.-
- net at Q2.2 (D): now also GROW2.1; no longer GROW2.+
- net at Q3.2 (D): now also GROW1.1; no longer GROW1.+
Changed lines of the file:
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@@
 		(on_board yes)
 		(dnp no)
-		(fields_autoplaced yes)
 		(property "Reference" "#PWR04"
 			(at 92.71 125.73 0)
@@
 		)
 		(property "Value" "+5V"
-			(at 92.71 116.84 0)
+			(at 95.504 119.888 0)
 			(effects
 				(font
@@
 	)
 	(symbol
+		(lib_name "HDSP-4840_1")
 		(lib_id "LED:HDSP-4840")
 		(at 45.72 129.54 270)
@@
 		(pin "12"
 		)
-		(pin "+"
+		(pin "1"
 		)
 		(pin "9"
@@
 		(pin "14"
 		)
-		(pin "-"
+		(pin "2"
 		)
 		(pin "16"
@@
 	)
 	(symbol
-		(lib_id "LED:HDSP-4840")
-		(at 92.71 127 270)
-		(unit 1)
-		(exclude_from_sim no)
-		(in_bom yes)
-		(on_board yes)
-		(dnp no)
-		(property "Reference" "GROW1"
-			(at 89.662 127 0)
-			(effects
-				(font
-					(size 1.27 1.27)
-				)
-			)
-		)
-		(property "Value" "~"
-			(at 96.52 127 0)
-			(effects
-				(font
-					(size 1.27 1.27)
-				)
-			)
-		)
-		(property "Footprint" "TerminalBlock_Phoenix:TerminalBlock_Phoenix_PT-1,5-2-3.5-H_1x02_P3.50mm_Horizontal"
-			(at 85.09 127 0)
-			(effects
-				(font
-					(size 1.27 1.27)
-				)
-				(hide yes)
-			)
-		)
-		(property "Datasheet" "https://www.amazon.com/Briignite-Spectrum-Strips-Indoor-Dimmable/dp/B0CH9Z5NW3?ref_=ast_sto_dp&th=1"
-			(at 92.71 127 0)
-			(effects
-				(font
-					(size 1.27 1.27)
-				)
-				(hide yes)
-			)
-		)
-		(property "Description" "Plant Grow Light Strip, Briignite Full Spectrum Grow Light Strips for Indoor Plants,15W LED Grow Light"
-			(at 92.71 127 0)
-			(effects
-				(font
-					(size 1.27 1.27)
-				)
-				(hide yes)
-			)
-		)
-		(property "Field5" ""
-			(at 92.71 127 0)
-			(effects
-				(font
-					(size 1.27 1.27)
-				)
-				(hide yes)
-			)
-		)
-		(pin "17"
-		)
-		(pin "13"
-		)
-		(pin "11"
-		)
-		(pin "2"
-		)
-		(pin "19"
-		)
-		(pin "3"
-		)
-		(pin "5"
-		)
-		(pin "12"
-		)
-		(pin "+"
-		)
-		(pin "9"
-		)
-		(pin "6"
-		)
-		(pin "14"
-		)
-		(pin "-"
-		)
-		(pin "16"
-		)
-		(pin "4"
-		)
-		(pin "18"
-		)
-		(pin "15"
-		)
-		(pin "8"
-		)
-		(pin "10"
-		)
-		(pin "7"
-		)
-		(instances
-			(project "Simple_Sprouts_PCB"
-				(path "/a5df5b5c-9e14-4fe1-8dcb-bdc183e40462"
-					(reference "GROW1")
-					(unit 1)
-				)
-			)
-		)
-	)
-	(symbol
 		(lib_id "Transistor_FET:IRLZ34N")
 		(at 46.99 99.06 0)
@@
 					(unit 1)
 				)
+			)
+		)
+	)
+	(symbol
+		(lib_name "HDSP-4840_1")
+		(lib_id "LED:HDSP-4840")
+		(at 92.71 127 270)
+		(unit 1)
+		(exclude_from_sim no)
+		(in_bom yes)
+		(on_board yes)
+		(dnp no)
+		(property "Reference" "GROW1"
+			(at 89.662 126.746 0)
+			(effects
+				(font
+					(size 1.27 1.27)
+				)
+			)
+		)
+		(property "Value" "~"
+			(at 96.52 127 0)
+			(effects
+				(font
+					(size 1.27 1.27)
+				)
+			)
+		)
+		(property "Footprint" "TerminalBlock_Phoenix:TerminalBlock_Phoenix_PT-1,5-2-3.5-H_1x02_P3.50mm_Horizontal"
+			(at 85.09 127 0)
+			(effects
+				(font
+					(size 1.27 1.27)
+				)
+				(hide yes)
+			)
+		)
+		(property "Datasheet" "https://www.amazon.com/Briignite-Spectrum-Strips-Indoor-Dimmable/dp/B0CH9Z5NW3?ref_=ast_sto_dp&th=1"
+			(at 92.71 127 0)
+			(effects
+				(font
+					(size 1.27 1.27)
+				)
+				(hide yes)
+			)
+		)
+		(property "Description" "Plant Grow Light Strip, Briignite Full Spectrum Grow Light Strips for Indoor Plants,15W LED Grow Light"
+			(at 92.71 127 0)
+			(effects
+				(font
+					(size 1.27 1.27)
+				)
+				(hide yes)
+			)
+		)
+		(pin "17"
+		)
+		(pin "13"
+		)
+		(pin "11"
+		)
+		(pin "2"
+		)
+		(pin "19"
+		)
+		(pin "3"
+		)
+		(pin "5"
+		)
+		(pin "12"
+		)
+		(pin "1"
+		)
+		(pin "9"
+		)
+		(pin "6"
+		)
+		(pin "14"
+		)
+		(pin "2"
+		)
+		(pin "16"
+		)
+		(pin "4"
+		)
+		(pin "18"
+		)
+		(pin "15"
+		)
+		(pin "8"
+		)
+		(pin "10"
+		)
+		(pin "7"
+		)
+		(instances
+			(project "Simple_Sprouts_PCB"
+				(path "/a5df5b5c-9e14-4fe1-8dcb-bdc183e40462"
+					(reference "GROW1")
+					(unit 1)
+				)

Commit message: Add files via upload
Parts:
- removed J2: 12V IN, Connector_PinHeader_2.00mm:PinHeader_1x01_P2.00mm_Vertical, symbol Connector_Generic:Conn_01x01
- removed J5: 5V IN, Connector_PinHeader_2.00mm:PinHeader_1x01_P2.00mm_Vertical, symbol Connector_Generic:Conn_01x01
- added 12V_IN1, 5V_IN1: Conn_01x02, TerminalBlock_Phoenix:TerminalBlock_Phoenix_PT-1,5-2-3.5-H_1x02_P3.50mm_Horizontal, symbol Connector_Generic:Conn_01x02
- R10, R11, R12, R13, R2, R3: footprint Resistor_SMD:R_0805_2012Metric -> Resistor_SMD:R_1206_3216Metric
- R14: footprint Resistor_SMD:R_1210_3225Metric -> Resistor_SMD:R_1206_3216Metric
- R15: footprint Resistor_SMD:R_2512_6332Metric -> Resistor_SMD:R_1206_3216Metric
Connections:
- net +12V: now also 12V_IN1.1 (Pin_1)
- net +5V: now also 5V_IN1.1 (Pin_1)
- net GND: now also 12V_IN1.2 (Pin_2), 5V_IN1.2 (Pin_2)
