File: PCB/Simple_Sprouts_PCB/Simple_Sprouts_PCB.kicad_pcb (KiCad board)
At the start: 2 copper layers, 100 x 100 mm, 29 parts, among them J1 Raspberry_Pi_5, Q1 IRLB8721PbF, Q2 IRLB8721PbF, Q3 IRLB8721PbF, Q4 IRLB8721PbF, Q5 IRLB8721PbF, Q6 IRLB8721PbF

Commit message: Add files via upload
Parts:
- J1: value Raspberry_Pi_5 -> Simple Sprouts PCB
- moved Q5 134.7 mm to (180.4, 89.5)
- moved Q2 132.7 mm to (180.4, 143.4)
- moved Q6 131.0 mm to (180.4, 110.5)
- moved Q4 130.9 mm to (180.4, 99.5)
- moved Q1 129.8 mm to (180.4, 121.5)
- moved Q3 129.6 mm to (180.4, 132.5)
- moved D7 123.8 mm to (193.5, 130.7), turned to -90 degrees
- moved D6 123.5 mm to (193.5, 96.7), turned to -90 degrees
- moved D5 122.9 mm to (193.5, 107.7), turned to -90 degrees
- moved D8 122.8 mm to (193.5, 118.7), turned to -90 degrees
- moved R6 100.4 mm to (172.5, 142.5), turned to 180 degrees
- moved D2 99.6 mm to (159.0, 88.5), turned to 180 degrees
- moved R5 98.1 mm to (172.5, 131.5), turned to 180 degrees
- moved D4 98.1 mm to (159.0, 109.5), turned to 180 degrees
- moved D1 97.2 mm to (159.0, 98.5), turned to 180 degrees
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Routing:
- added copper zone on In1.Cu, net GND
Other:
- board size 100 x 100 mm -> 59 x 66.5 mm
- copper layers 2 -> 4

Commit message: Add files via upload
Parts:
- J1: footprint RASPBERRY_PI_4B_4GB:MODULE_RASPBERRY_PI_4B_4GB -> RASPBERRY_PI_4B_4GB:Pin_Replacement
- moved J1 52.9 mm to (120.9, 72.3), turned to 0 degrees
- moved R6 51.9 mm to (130.3, 112.3), turned to -90 degrees
- moved R5 50.2 mm to (130.3, 104.3), turned to -90 degrees
- moved R7 48.4 mm to (130.3, 96.3), turned to -90 degrees
- moved D7 47.9 mm to (156.3, 100.5)
- moved D5 47.3 mm to (156.3, 78.5)
- moved D6 47.3 mm to (156.3, 67.5)
- moved D8 47.3 mm to (156.3, 89.5)
- moved R9 47.0 mm to (130.3, 88.3), turned to -90 degrees
- moved R8 45.8 mm to (130.3, 80.3), turned to -90 degrees
- moved R4 45.0 mm to (130.3, 72.3), turned to -90 degrees
- moved Q3 44.7 mm to (142.2, 109.3)
- moved Q2 44.7 mm to (142.2, 120.3)
- moved Q1 44.2 mm to (142.2, 99.3)
- moved Q4 44.2 mm to (142.2, 77.3)
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Connections:
- J1 pad 11: unconnected-(J1-GPIO17/SPI1_~{CE1}-Pad11) -> Net-(J1-GPIO17/SPI1_~{CE1})
- J1 pad 15: unconnected-(J1-GPIO22/SDIO_CLK-Pad15) -> Net-(J1-GPIO22/SDIO_CLK)
- J1 pad 16: unconnected-(J1-GPIO23/SDIO_CMD-Pad16) -> Net-(J1-GPIO23/SDIO_CMD)
- J1 pad 19: unconnected-(J1-MOSI_SPI0/GPIO10-Pad19) -> Net-(J1-MOSI_SPI0/GPIO10)
- J1 pad 22: Net-(J1-GPIO25/SDIO_DAT1) -> unconnected-(J1-GPIO25/SDIO_DAT1-Pad22)
- J1 pad 23: Net-(J1-SCLK_SPI0/GPIO11) -> unconnected-(J1-SCLK_SPI0/GPIO11-Pad23)
- J1 pad 27: unconnected-(J1-ID_SD_I2C0/GPIO00-Pad27) -> Net-(J1-ID_SD_I2C0/GPIO00)
- J1 pad 29: Net-(J1-GPCLK1/GPIO05) -> unconnected-(J1-GPCLK1/GPIO05-Pad29)
- J1 pad 32: Net-(J1-GPIO12/PWM0) -> unconnected-(J1-GPIO12/PWM0-Pad32)
- J1 pad 35: unconnected-(J1-GPIO19/SPI1_MISO/PCM_FS-Pad35) -> Net-(J1-GPIO19/SPI1_MISO/PCM_FS)
- J1 pad 37: Net-(J1-GPIO26/SDIO_DAT2) -> unconnected-(J1-GPIO26/SDIO_DAT2-Pad37)
- J1 pad 7: Net-(J1-GPCLK0/GPIO04) -> unconnected-(J1-GPCLK0/GPIO04-Pad7)
- Q1 pad 1: Net-(J1-GPIO27/SDIO_DAT3) -> Net-(J1-MOSI_SPI0/GPIO10)
- Q2 pad 1: Net-(J1-GPIO26/SDIO_DAT2) -> Net-(J1-GPIO17/SPI1_~{CE1})
- Q3 pad 1: Net-(J1-GPIO25/SDIO_DAT1) -> Net-(J1-GPIO22/SDIO_CLK)
- Q4 pad 1: Net-(J1-GPIO12/PWM0) -> Net-(J1-GPIO13/PWM1)
- Q5 pad 1: Net-(J1-GPIO13/PWM1) -> Net-(J1-GPIO19/SPI1_MISO/PCM_FS)
- Q6 pad 1: Net-(J1-SCLK_SPI0/GPIO11) -> Net-(J1-ID_SD_I2C0/GPIO00)
- R14 pad 1: Net-(J1-GPCLK1/GPIO05) -> Net-(J1-GPIO27/SDIO_DAT3)
- R15 pad 1: Net-(J1-GPCLK1/GPIO05) -> Net-(J1-GPIO27/SDIO_DAT3)
- R4 pad 1: Net-(J1-GPIO13/PWM1) -> Net-(J1-GPIO19/SPI1_MISO/PCM_FS)
- R5 pad 1: Net-(J1-GPIO25/SDIO_DAT1) -> Net-(J1-GPIO22/SDIO_CLK)
- R6 pad 1: Net-(J1-GPIO26/SDIO_DAT2) -> Net-(J1-GPIO17/SPI1_~{CE1})
- R7 pad 1: Net-(J1-GPIO27/SDIO_DAT3) -> Net-(J1-MOSI_SPI0/GPIO10)
- R8 pad 1: Net-(J1-GPIO12/PWM0) -> Net-(J1-GPIO13/PWM1)
- R9 pad 1: Net-(J1-SCLK_SPI0/GPIO11) -> Net-(J1-ID_SD_I2C0/GPIO00)
Routing:
- net GND: track 0.00 -> 150.4 mm, vias 0 -> 7
- net +12V: track 0.00 -> 98.4 mm, vias 0 -> 4
- net Net-(J1-GPIO27/SDIO_DAT3): track 0.00 -> 44.8 mm
- net Net-(J1-GPIO17/SPI1_~{CE1}): track 0.00 -> 25.3 mm
- net Net-(D6-K): track 0.00 -> 24.3 mm
- net Net-(D5-K): track 0.00 -> 23.2 mm
- net Net-(J1-GPIO22/SDIO_CLK): track 0.00 -> 23.0 mm
- net Net-(D8-K): track 0.00 -> 22.2 mm
- net Net-(D7-K): track 0.00 -> 21.8 mm
- net Net-(J1-GPIO19/SPI1_MISO/PCM_FS): track 0.00 -> 20.9 mm
- net Net-(J1-MOSI_SPI0/GPIO10): track 0.00 -> 19.8 mm
- net Net-(J1-ID_SD_I2C0/GPIO00): track 0.00 -> 18.8 mm
- net Net-(J1-GPIO13/PWM1): track 0.00 -> 18.7 mm
- net Net-(J1-SCL_I2C1/GPIO03): track 0.00 -> 12.2 mm
- net +3.3V: track 0.00 -> 11.1 mm, vias 0 -> 2
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- added copper zone on In2.Cu, net +12V
- added copper zone on In2.Cu, net +3.3V
Other:
- board size 59 x 66.5 mm -> 56 x 66.5 mm

Commit message: Add files via upload
Parts:
- removed J1: Simple Sprouts PCB, RASPBERRY_PI_4B_4GB:Pin_Replacement
- added REF**: Pin_Replacement, RASPBERRY_PI_4B_4GB:Pin_Replacement, F.Cu at (120.9, 72.3)
- added T. Block: TerminalBlock_Phoenix_MKDS-1,5-2_1x02_P5.00mm_Horizontal, TerminalBlock_Phoenix:TerminalBlock_Phoenix_MKDS-1,5-2_1x02_P5.00mm_Horizontal, F.Cu at (167.1, 116.5)
- R4, R5, R6, R7, R8, R9: value 220Ω -> 10kΩ
- moved R14 7.82 mm to (159.0, 119.9), turned to -90 degrees
- moved R15 4.01 mm to (154.3, 117.2)
Connections:
- D5 pad 1: Net-(D5-K) -> +12V
- D5 pad 2: +12V -> Net-(D5-A)
- D6 pad 1: Net-(D6-K) -> +12V
- D6 pad 2: +12V -> Net-(D6-A)
- D7 pad 1: Net-(D7-K) -> +12V
- D7 pad 2: +12V -> Net-(D7-A)
- D8 pad 1: Net-(D8-K) -> +12V
- D8 pad 2: +12V -> Net-(D8-A)
- Q1 pad 2: Net-(D7-K) -> Net-(D7-A)
- Q4 pad 2: Net-(D5-K) -> Net-(D5-A)
- Q5 pad 2: Net-(D6-K) -> Net-(D6-A)
- Q6 pad 2: Net-(D8-K) -> Net-(D8-A)
- R10 pad 2: Net-(D5-K) -> Net-(D5-A)
- R11 pad 2: Net-(D6-K) -> Net-(D6-A)
- R12 pad 2: Net-(D7-K) -> Net-(D7-A)
- R13 pad 2: Net-(D8-K) -> Net-(D8-A)
Routing:
- net +12V: track 98.4 -> 136.2 mm
- net Net-(D6-K): track 24.3 -> 0.00 mm
- net Net-(D5-K): track 23.2 -> 0.00 mm
- net Net-(D5-A): track 0.00 -> 22.4 mm
- net Net-(D8-K): track 22.2 -> 0.00 mm
- net Net-(D6-A): track 0.00 -> 22.1 mm
- net Net-(D7-K): track 21.8 -> 0.00 mm
- net Net-(D8-A): track 0.00 -> 21.1 mm
- net Net-(D7-A): track 0.00 -> 20.7 mm
- net Net-(J1-GPIO27/SDIO_DAT3): track 44.8 -> 40.8 mm
- net GND: track 150.4 -> 146.9 mm

Commit message: Add files via upload
Other:
- board size 56 x 66.5 mm -> 58 x 66.5 mm
Changed lines of the file:
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@@
 	)
 	(gr_rect
-		(start 119.27 60.8)
-		(end 175.27 127.3)
+		(start 118.27 60.8)
+		(end 176.27 127.3)
 		(stroke
 			(width 0.05)
@@
 	(segment
 		(start 130.27 73.7625)
-		(end 128.641638 73.7625)
+		(end 129.7625 73.7625)
 		(width 2)
 		(layer "In1.Cu")
@@
 	)
 	(segment
-		(start 128.641638 73.7625)
-		(end 124.649138 69.77)
-		(width 2)
-		(layer "In1.Cu")
-		(net 10)
-	)
-	(segment
 		(start 133.7325 70.3)
 		(end 130.27 73.7625)
@@
 	)
 	(segment
-		(start 124.649138 69.77)
-		(end 124.29 69.77)
-		(width 2)
-		(layer "In1.Cu")
-		(net 10)
-	)
-	(segment
 		(start 130.27 113.7625)
 		(end 130.27 105.7625)
@@
 	)
 	(segment
+		(start 125.77 69.77)
+		(end 124.29 69.77)
+		(width 2)
+		(layer "In1.Cu")
+		(net 10)
+	)
+	(segment
 		(start 147.27 68.3)
 		(end 145.77 69.8)
@@
 		(start 145.77 69.8)
 		(end 145.27 70.3)
+		(width 2)
+		(layer "In1.Cu")
+		(net 10)
+	)
+	(segment
+		(start 129.7625 73.7625)
+		(end 125.77 69.77)
 		(width 2)
 		(layer "In1.Cu")
@@
 		(polygon
 			(pts
-				(xy 119.27 127.3) (xy 169.27 127.3) (xy 175.27 127.3) (xy 175.27 61.3) (xy 169.27 61.3) (xy 132.27 61.3)
-				(xy 119.27 61.3)
+				(xy 118.27 127.3) (xy 169.27 127.3) (xy 176.27 127.3) (xy 176.27 61.3) (xy 169.27 61.3) (xy 132.27 61.3)
+				(xy 118.27 61.3)
 			)
 		)
@@
 		(polygon
 			(pts
-				(xy 151.27 61.3) (xy 151.27 108.3) (xy 175.27 108.3) (xy 175.27 61.3)
+				(xy 151.27 61.3) (xy 151.27 108.3) (xy 176.27 108.3) (xy 176.27 61.3)
 			)
 		)

Commit message: Add files via upload
Parts:
- removed REF**: Pin_Replacement, RASPBERRY_PI_4B_4GB:Pin_Replacement
- removed T. Block: TerminalBlock_Phoenix_MKDS-1,5-2_1x02_P5.00mm_Horizontal, TerminalBlock_Phoenix:TerminalBlock_Phoenix_MKDS-1,5-2_1x02_P5.00mm_Horizontal
- added J1: Raspberry_Pi_5, RASPBERRY_PI_4B_4GB:Pin_Replacement, F.Cu at (120.9, 72.3)
- added J3: Soil Sensor, Connector_PinHeader_2.54mm:PinHeader_1x04_P2.54mm_Vertical, F.Cu at (60.0, 154.9)
- added J4: Soil Sensor, Connector_PinHeader_2.54mm:PinHeader_1x04_P2.54mm_Vertical, F.Cu at (77.0, 155.2)
- added J6: Temperature Sensor, Connector_PinHeader_2.54mm:PinHeader_1x04_P2.54mm_Vertical, F.Cu at (91.5, 158.0)
- added J7: Air Quality Sensor, Connector_PinHeader_2.54mm:PinHeader_1x04_P2.54mm_Vertical, F.Cu at (109.0, 175.0)
- added J8: Humidity Sensor, Connector_PinHeader_2.54mm:PinHeader_1x04_P2.54mm_Vertical, F.Cu at (142.0, 172.4)
- added J9: Distance Sensor, Connector_PinHeader_2.54mm:PinHeader_1x04_P2.54mm_Vertical, F.Cu at (98.5, 129.9)
- added LEDStrip1: ~, TerminalBlock_Phoenix:TerminalBlock_Phoenix_MPT-0,5-2-2.54_1x02_P2.54mm_Horizontal, F.Cu at (18.7, 112.5)
- added LEDStrip2: ~, TerminalBlock_Phoenix:TerminalBlock_Phoenix_MPT-0,5-2-2.54_1x02_P2.54mm_Horizontal, F.Cu at (21.2, 144.5)
- added R1: Heater Module, TerminalBlock_Phoenix:TerminalBlock_Phoenix_MPT-0,5-2-2.54_1x02_P2.54mm_Horizontal, F.Cu at (34.2, 168.5)
- added Solenoid_Valve1: L, TerminalBlock_Phoenix:TerminalBlock_Phoenix_MPT-0,5-2-2.54_1x02_P2.54mm_Horizontal, F.Cu at (57.2, 180.5)
- added Solenoid_Valve2: L, TerminalBlock_Phoenix:TerminalBlock_Phoenix_MPT-0,5-2-2.54_1x02_P2.54mm_Horizontal, F.Cu at (84.2, 188.5)
- added WaterPump: 12V, TerminalBlock_Phoenix:TerminalBlock_Phoenix_MPT-0,5-2-2.54_1x02_P2.54mm_Horizontal, F.Cu at (67.9, 131.7)
- moved R14 4.87 mm to (162.7, 116.7)
- moved R15 1.07 mm to (155.3, 117.2)
Routing:
- net Net-(J1-GPIO27/SDIO_DAT3): track 40.8 -> 44.4 mm
- net Net-(D8-A): track 21.1 -> 22.5 mm
- net Net-(D7-A): track 20.7 -> 22.1 mm
- net GND: track 146.9 -> 148.1 mm
- net Net-(D5-A): track 22.4 -> 23.3 mm
- net Net-(D6-A): track 22.1 -> 23.0 mm
Other:
- board size 58 x 66.5 mm -> 58 x 99.5 mm

Commit message: Add files via upload
Parts:
- moved LEDStrip2 163.5 mm to (181.8, 114.2), turned to 90 degrees
- moved R1 161.1 mm to (181.8, 103.8), turned to 180 degrees
- moved Solenoid_Valve1 160.1 mm to (181.8, 80.0), turned to 180 degrees
- moved Solenoid_Valve2 154.7 mm to (181.8, 68.5), turned to 180 degrees
- moved LEDStrip1 153.5 mm to (172.2, 114.2), turned to 90 degrees
- moved J3 128.9 mm to (184.2, 120.5)
- moved WaterPump 120.5 mm to (181.8, 92.4), turned to 180 degrees
- moved J7 89.0 mm to (179.2, 120.3)
- moved J6 74.3 mm to (159.0, 126.7), turned to 90 degrees
- moved J9 67.1 mm to (165.0, 120.2), turned to -90 degrees
- moved J4 59.1 mm to (129.1, 127.2), turned to 90 degrees
- moved J8 45.4 mm to (144.1, 127.0), turned to 90 degrees
- moved R14 10.2 mm to (152.5, 116.2)
- moved R15 6.16 mm to (160.5, 113.8), turned to 0 degrees
Connections:
- J9 pad 3: Net-(J9-Pin_3) -> Net-(J1-GPIO27/SDIO_DAT3)
- LEDStrip1 pad 1: (no net) -> Net-(Q3-D)
- LEDStrip1 pad 2: (no net) -> +5V
- LEDStrip2 pad 1: (no net) -> Net-(Q2-D)
- LEDStrip2 pad 2: (no net) -> +5V
- R14 pad 2: Net-(J9-Pin_3) -> Net-(J1-GPIO27/SDIO_DAT3)
Routing:
- net GND: track 148.1 -> 270.1 mm
- net Net-(J1-SCL_I2C1/GPIO03): track 12.2 -> 112.9 mm
- net +5V: track 0.00 -> 81.1 mm
- net Net-(J1-SDA_I2C1/GPIO02): track 6.14 -> 81.2 mm
- net +12V: track 136.2 -> 200.2 mm
- net Net-(J1-GPIO23/SDIO_CMD): track 0.00 -> 53.5 mm
- net Net-(Q2-D): track 0.00 -> 45.4 mm
- net Net-(D7-A): track 22.1 -> 63.9 mm
- net Net-(D6-A): track 23.0 -> 63.7 mm
- net Net-(D8-A): track 22.5 -> 62.7 mm
- net Net-(D5-A): track 23.3 -> 62.8 mm
- net Net-(Q3-D): track 0.00 -> 32.6 mm
- net Net-(J1-GPIO27/SDIO_DAT3): track 44.4 -> 47.2 mm
- added copper zone on In2.Cu, net +5V
Other:
- board size 58 x 99.5 mm -> 69 x 70.6 mm

Commit message: Add files via upload
Parts:
- added 12V IN: 12V IN, Connector_PinHeader_2.00mm:PinHeader_1x01_P2.00mm_Vertical, F.Cu at (131.3, 64.2)
- added 5V IN: 5V IN, Connector_PinHeader_2.00mm:PinHeader_1x01_P2.00mm_Vertical, F.Cu at (161.5, 109.5)
- J1: footprint RASPBERRY_PI_4B_4GB:Pin_Replacement -> RASPBERRY_PI_4B_4GB:RPI Pins
- J9: value Distance Sensor -> HC-SR04
- R1: value Heater Module -> Heater
- Water Pump: renamed from WaterPump
- renumbered LEDStrip1 to GROW1, LEDStrip2 to GROW2, Solenoid_Valve1 to Valve1, Solenoid_Valve2 to Valve2
Connections:
- GROW1 pad 1: Net-(Q3-D) -> (no net)
- GROW1 pad 2: +5V -> (no net)
- GROW2 pad 1: Net-(Q2-D) -> (no net)
- GROW2 pad 2: +5V -> (no net)
- J9 pad 3: Net-(J1-GPIO27/SDIO_DAT3) -> Net-(J9-Pin_3)
- R14 pad 2: Net-(J1-GPIO27/SDIO_DAT3) -> Net-(J9-Pin_3)
Routing:
- net +12V: track 200.2 -> 237.0 mm
- net +5V: track 81.1 -> 92.3 mm
- net Net-(J1-GPIO27/SDIO_DAT3): track 47.2 -> 38.6 mm
- net Net-(J9-Pin_3): track 0.00 -> 8.60 mm

Commit message: Add files via upload
Connections:
- GROW1 pad 1: (no net) -> Net-(Q3-D)
- GROW1 pad 2: (no net) -> +5V
- GROW2 pad 1: (no net) -> Net-(Q2-D)
- GROW2 pad 2: (no net) -> +5V
Routing:
- net +3.3V: track 11.1 -> 34.4 mm
- net +5V: track 92.3 -> 113.9 mm
- net Net-(Q2-D): track 45.4 -> 44.3 mm
- net Net-(D5-A): track 62.8 -> 62.0 mm
- removed copper zone on In2.Cu, net +3.3V
Changed lines of the file:
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@@
 			(layers "*.Cu" "*.Mask")
 			(remove_unused_layers no)
+			(net 18 "Net-(Q3-D)")
 		)
 		(pad "2" thru_hole circle
@@
 			(layers "*.Cu" "*.Mask")
 			(remove_unused_layers no)
+			(net 11 "+5V")
 		)
 		(model "${KICAD8_3DMODEL_DIR}/TerminalBlock_Phoenix.3dshapes/TerminalBlock_Phoenix_MPT-0,5-2-2.54_1x02_P2.54mm_Horizontal.wrl"
@@
 			(at 2.11 48.25 180)
 			(layer "F.SilkS")
+			(hide yes)
 			(effects
 				(font
@@
 			(layers "*.Cu" "*.Mask")
 			(remove_unused_layers no)
+			(net 17 "Net-(Q2-D)")
 		)
 		(pad "2" thru_hole circle
@@
 			(layers "*.Cu" "*.Mask")
 			(remove_unused_layers no)
+			(net 11 "+5V")
 		)
 		(model "${KICAD8_3DMODEL_DIR}/TerminalBlock_Phoenix.3dshapes/TerminalBlock_Phoenix_MPT-0,5-2-2.54_1x02_P2.54mm_Horizontal.wrl"
@@
 	)
 	(segment
-		(start 163.445 84.3)
-		(end 163.445 83.475)
-		(width 0.2)
-		(layer "F.Cu")
-		(net 6)
-	)
-	(segment
 		(start 164.47 79.97)
 		(end 179.25 79.97)
@@
 	)
 	(segment
+		(start 119.09 120.72)
+		(end 121.74 118.07)
+		(width 1)
+		(layer "In2.Cu")
+		(net 11)
+	)
+	(segment
 		(start 159 124.5)
 		(end 163.73 124.5)
@@
 	)
 	(segment
+		(start 129.08 127.17)
+		(end 120.96 127.17)
+		(width 1)
+		(layer "In2.Cu")
+		(net 11)
+	)
+	(segment
 		(start 179.74 109.5)
 		(end 181.85 111.61)
@@
 	)
 	(segment
+		(start 119.09 125.3)
+		(end 119.09 120.72)
+		(width 1)
+		(layer "In2.Cu")
+		(net 11)
+	)
+	(segment
 		(start 158.96 126.71)
 		(end 156.17 129.5)
@@
 	)
 	(segment
+		(start 120.96 127.17)
+		(end 119.09 125.3)
+		(width 1)
+		(layer "In2.Cu")
+		(net 11)
+	)
+	(segment
 		(start 179.21 120.3)
 		(end 183.96 120.3)
@@
 	)
 	(segment
+		(start 121.74 118.07)
+		(end 121.74 115.53)
+		(width 1)
+		(layer "In2.Cu")
+		(net 11)
+	)
+	(segment
 		(start 164.96 123.27)
 		(end 164.96 120.42)
@@
 	)
 	(segment
-		(start 126.575 118.43)
-		(end 129.27 121.125)
+		(start 129.125 121.125)
+		(end 125.75 117.75)
+		(width 0.2)
+		(layer "In2.Cu")
+		(net 12)
+	)
+	(segment
+		(start 124.28 97.75)
+		(end 126.75 100.22)
+		(width 0.2)
+		(layer "In2.Cu")
+		(net 12)
+	)
+	(segment
+		(start 126.75 116)
+		(end 124.68 118.07)
+		(width 0.2)
+		(layer "In2.Cu")
+		(net 12)
+	)
+	(segment
+		(start 129.27 121.125)
+		(end 129.5 121.125)
 		(width 0.2)
 		(layer "In2.Cu")
@@
 	)
 	(segment
-		(start 124.54 118.43)
-		(end 126.575 118.43)
+		(start 125.75 117.75)
+		(end 124.6 117.75)
 		(width 0.2)
 		(layer "In2.Cu")
@@
 	(segment
 		(start 129.27 121.125)
+		(end 129.125 121.125)
+		(width 0.2)
+		(layer "In2.Cu")
+		(net 12)
+	)
+	(segment
+		(start 124.6 117.75)
+		(end 124.28 118.07)
+		(width 0.2)
+		(layer "In2.Cu")
+		(net 12)
+	)
+	(segment
+		(start 129.5 121.125)
 		(end 134.27 121.125)
 		(width 0.2)
@@
 	)
 	(segment
+		(start 124.68 118.07)
+		(end 124.28 118.07)
+		(width 0.2)
+		(layer "In2.Cu")
+		(net 12)
+	)
+	(segment
+		(start 126.75 100.22)
+		(end 126.75 116)
+		(width 0.2)
+		(layer "In2.Cu")
+		(net 12)
+	)
+	(segment
 		(start 134.16 124.46)
 		(end 134.17 124.45)
@@
 	)
 	(segment
-		(start 180.77 114.15)
-		(end 181.85 114.15)
-		(width 0.2)
-		(layer "F.Cu")
-		(net 17)
-	)
-	(segment
-		(start 178.75 117.25)
-		(end 181.85 114.15)
+		(start 171.668881 117.25)
+		(end 178.75 117.25)
 		(width 2)
 		(layer "F.Cu")
@@
 	)
 	(segment
-		(start 171.668881 117.25)
-		(end 178.75 117.25)
+		(start 167.5 123.15)
+		(end 167.5 121.418881)
 		(width 2)
 		(layer "F.Cu")
@@
 	)
 	(segment
-		(start 167.5 123.15)
-		(end 167.5 121.418881)
+		(start 178.75 117.25)
+		(end 181.85 114.15)
 		(width 2)
 		(layer "F.Cu")
@@
 	)
 	(segment
+		(start 170.71 114.21)
+		(end 172.21 114.21)
+		(width 2)
+		(layer "F.Cu")
+		(net 18)
+	)
+	(segment
 		(start 165 107)
 		(end 166 108)
@@
 	)
 	(segment
-		(start 170.71 114.21)
-		(end 172.21 114.21)
-		(width 2)
-		(layer "F.Cu")
-		(net 18)
-	)
-	(segment
 		(start 129.8075 86.8375)
 		(end 128.38 85.41)
@@
 		(polygon
 			(pts
-				(xy 122.5 117) (xy 122.5 119.5) (xy 119.53 119.49) (xy 119.53 126.49) (xy 126 126.5) (xy 126 125)
+				(xy 122.5 114.5) (xy 122.5 119.5) (xy 119.53 119.49) (xy 119.53 126.49) (xy 126 126.5) (xy 126 125)
 				(xy 156 125) (xy 156 123) (xy 163.22 123.02) (xy 163.22 114.02) (xy 167.5 114) (xy 167.5 108.5)
-				(xy 186 108.5) (xy 186 130.5) (xy 118.81 130.44) (xy 118.81 116.94)
-			)
-		)
-	)
-	(zone
-		(net 12)
-		(net_name "+3.3V")
-		(layer "In2.Cu")
-		(hatch edge 0.5)
-		(priority 1)
-		(connect_pads
-			(clearance 0.5)
-		)
-		(min_thickness 0.25)
-		(filled_areas_thickness no)
-		(fill yes
-			(thermal_gap 0.5)
-			(thermal_bridge_width 0.5)
-			(smoothing chamfer)
-		)
-		(polygon
-			(pts
-				(xy 137.2 124.4) (xy 137.27 117.3) (xy 123.27 117.3) (xy 123.47 124.3)
+				(xy 186 108.5) (xy 186 130.5) (xy 118.81 130.44) (xy 118.81 114.44)
 			)
 		)
