File: PCB/Simple_Sprouts_PCB/Simple_Sprouts_PCB.kicad_pcb (KiCad board)
At the start: 4 copper layers, 69 x 70.6 mm, 43 parts, among them J1 Raspberry_Pi_5, J3 Soil Sensor, J4 Soil Sensor, J6 Temperature Sensor, J7 Air Quality Sensor, J8 Humidity Sensor, J9 HC-SR04, Q1 IRLB8721PbF, Q2 IRLB8721PbF, Q3 IRLB8721PbF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

Commit message: Add files via upload
Parts:
- D1, D2, D3, D4: footprint my-LED-4mm-3mm:LED_D4.0mm_P3.0mm -> LED_THT:LED_D5.0mm
- D5, D6, D7, D8: footprint Diode_SMD:D_SMB -> Diode_SMD:D_SMA
- GROW1, GROW2, Valve1, Valve2: footprint TerminalBlock_Phoenix:TerminalBlock_Phoenix_MPT-0,5-2-2.54_1x02_P2.54mm_Horizontal -> TerminalBlock_Phoenix:TerminalBlock_Phoenix_PT-1,5-2-3.5-H_1x02_P3.50mm_Horizontal
- J1: footprint RASPBERRY_PI_4B_4GB:RPI Pins -> RASPBERRY_PI_4B_4GB:RPI Correct
- J12: renamed from Water Pump; footprint TerminalBlock_Phoenix:TerminalBlock_Phoenix_MPT-0,5-2-2.54_1x02_P2.54mm_Horizontal -> TerminalBlock_Phoenix:TerminalBlock_Phoenix_PT-1,5-2-3.5-H_1x02_P3.50mm_Horizontal
- J2: renamed from 12V IN
- J5: renamed from 5V IN
- R1: value Heater -> R1; footprint TerminalBlock_Phoenix:TerminalBlock_Phoenix_MPT-0,5-2-2.54_1x02_P2.54mm_Horizontal -> TerminalBlock_Phoenix:TerminalBlock_Phoenix_PT-1,5-2-3.5-H_1x02_P3.50mm_Horizontal
- R10, R11, R12, R13: value 5kΩ -> 1kΩ
- moved GROW1 1.12 mm to (171.1, 113.9)
- moved GROW2 0.39 mm to (181.5, 114.0)
Connections:
- GROW1 pad 1: Net-(Q3-D) -> (no net)
- GROW1 pad 2: +5V -> (no net)
- GROW2 pad 1: Net-(Q2-D) -> (no net)
- GROW2 pad 2: +5V -> (no net)
Routing:
- net +12V: track 237.0 -> 233.5 mm
- net Net-(D7-A): track 63.9 -> 62.9 mm
- net Net-(D6-A): track 63.7 -> 62.7 mm
- net Net-(D5-A): track 62.0 -> 61.0 mm
- net Net-(D8-A): track 62.7 -> 61.7 mm

Commit message: Add files via upload
Parts:
- moved GROW1 0.11 mm to (171.1, 114.0)
- moved GROW2 0.06 mm to (181.6, 114.0)
Connections:
- GROW1 pad 1: (no net) -> Net-(Q3-D)
- GROW1 pad 2: (no net) -> +5V
- GROW2 pad 1: (no net) -> Net-(Q2-D)
- GROW2 pad 2: (no net) -> +5V
Routing:
- net +5V: track 113.6 -> 110.9 mm
