File: PCB/Simple_Sprouts_PCB/Simple_Sprouts_PCB.kicad_pcb (KiCad board)
At the start: 4 copper layers, 69 x 70.6 mm, 43 parts, among them J1 Raspberry_Pi_5, J12 12V, J2 12V IN, J3 Soil Sensor, J4 Soil Sensor, J5 5V IN, J6 Temperature Sensor, J7 Air Quality Sensor, J8 Humidity Sensor, J9 HC-SR04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

Commit message: Add files via upload
Parts:
- removed J2: 12V IN, Connector_PinHeader_2.00mm:PinHeader_1x01_P2.00mm_Vertical
- removed J5: 5V IN, Connector_PinHeader_2.00mm:PinHeader_1x01_P2.00mm_Vertical
- added 12V IN: Conn_01x02, TerminalBlock_Phoenix:TerminalBlock_Phoenix_PT-1,5-2-3.5-H_1x02_P3.50mm_Horizontal, F.Cu at (133.8, 64.5)
- added 5V IN: Conn_01x02, TerminalBlock_Phoenix:TerminalBlock_Phoenix_PT-1,5-2-3.5-H_1x02_P3.50mm_Horizontal, F.Cu at (161.2, 113.2)
- R10, R11, R12, R13, R2, R3: footprint Resistor_SMD:R_0805_2012Metric -> Resistor_SMD:R_1206_3216Metric
- R14: footprint Resistor_SMD:R_1210_3225Metric -> Resistor_SMD:R_1206_3216Metric
- R15: footprint Resistor_SMD:R_2512_6332Metric -> Resistor_SMD:R_1206_3216Metric
- Water Pump: renamed from J12
- moved R15 8.56 mm to (152.5, 110.8), turned to 90 degrees
- moved Heater 1.94 mm to (180.8, 102.2), turned to 90 degrees
- moved GROW2 1.82 mm to (181.1, 112.2)
- moved GROW1 1.63 mm to (169.5, 113.5), turned to 0 degrees
- moved Water Pump 1.57 mm to (180.8, 91.2), turned to 90 degrees
- moved Valve1 1.30 mm to (180.8, 80.8), turned to 90 degrees
- moved Valve2 1.17 mm to (180.8, 69.0), turned to 90 degrees
- renumbered R1 to Heater
Routing:
- net GND: track 270.1 -> 295.9 mm
- net +12V: track 233.8 -> 212.3 mm
- net +5V: track 110.9 -> 115.6 mm
- net Net-(D6-A): track 62.7 -> 66.4 mm
- net Net-(D5-A): track 61.0 -> 64.6 mm
- net Net-(J1-GPIO27/SDIO_DAT3): track 38.6 -> 35.7 mm
- net Net-(D8-A): track 61.7 -> 64.1 mm
- net Net-(Q3-D): track 32.5 -> 30.8 mm
- net Net-(Q2-D): track 44.4 -> 46.0 mm
- net Net-(D7-A): track 62.9 -> 64.3 mm
Other:
- board size 69 x 70.6 mm -> 69 x 72.4 mm

Commit message: Add files via upload
Routing:
- net +12V: track 212.3 -> 21.3 mm
- net +5V: track 115.6 -> 29.3 mm
- net GND: track 295.9 -> 290.7 mm
